File: HARDWARE/Versión Taller/V.Normal.kicad_pcb (KiCad board)
At the start: 2 copper layers, 60.5 x 36.5 mm, 27 parts, among them J1 Ds18b20, J2 MPU-6050, J3 Max30102, J4 Conn_01x02_Pin, J5 BAT 3,7 3000 mAh, J6 USB, Q1 Q_NPN_BEC, Q2 MMBT2222A, SW1 SW_SPST, SW3 EN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

Commit message: Parte Final
Parts:
- SW3, SW4: footprint Button_Switch_SMD:SW_SPST_CK_RS282G05A3 -> Button_Switch_THT:SW_PUSH_1P1T_6x3.5mm_H5.0_APEM_MJTP1250; moved to B.Cu
- moved SW4 3.93 mm to (112.3, 78.2)
- moved SW3 3.93 mm to (100.1, 78.5)
- moved R2 0.54 mm to (122.5, 73.1)
- moved R3 0.53 mm to (117.5, 73.1)
Routing:
- net BOOT: track 21.7 -> 18.7 mm
- net +BATT: track 11.1 -> 11.6 mm
- net /IND.BAT: track 13.4 -> 12.8 mm
