File: HARDWARE/Versión Taller/V.Normal.kicad_sch (KiCad schematic)
At the start: 27 parts, among them J1 Ds18b20, J2 MPU-6050, J3 Max30102, J4 Conn_01x02_Pin, J5 IND.BAT 3,7 3000 mAh, J6 USB, Q1 Q_NPN_BEC, Q2 MMBT2222A, SW1 SW_SPST, SW3 EN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

Commit message: Parte Final
Parts:
- SW3, SW4: footprint Button_Switch_SMD:SW_SPST_CK_RS282G05A3 -> Button_Switch_THT:SW_PUSH_1P1T_6x3.5mm_H5.0_APEM_MJTP1250
Changed lines of the file:
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@@
 			)
 		)
-		(property "Footprint" "Button_Switch_SMD:SW_SPST_CK_RS282G05A3"
+		(property "Footprint" "Button_Switch_THT:SW_PUSH_1P1T_6x3.5mm_H5.0_APEM_MJTP1250"
 			(at 80.01 91.44 0)
 			(hide yes)
@@
 			)
 		)
-		(property "Footprint" "Button_Switch_SMD:SW_SPST_CK_RS282G05A3"
+		(property "Footprint" "Button_Switch_THT:SW_PUSH_1P1T_6x3.5mm_H5.0_APEM_MJTP1250"
 			(at 80.01 78.74 0)
 			(hide yes)
